File: sensor/kicad/kicad.kicad_sch (KiCad schematic)
At the start: 14 parts, among them J1 MQ-135, J2 DHT11, J3 LM-393, J4 MSM261, U1 ESP32-S3-WROOM-1

Commit message: scheme
Parts:
- removed R5, R6, R7: R, symbol Device:R
- D1: value LED -> LED Y
- D2: value LED -> LED G
- D3: value LED -> LED R
- R3: renamed from R4; value R -> 1k
Connections:
- net GND: now also R3.2
- net at D1.1 (K): now also D2.1 (K), D3.1 (K), R3.1
- net at D1.2 (A): now also U1.10 (IO17)
- net at J4.2 (SD): now also U1.21 (IO13)
- net at J4.3 (SCK): now also U1.22 (IO14)
- net at J4.4 (WS): now also U1.8 (IO15)
- net at D2.2 (A): now also U1.11 (IO18)
- net at U1.9 (IO16): now also D3.2 (A)
Other:
- moved on the sheet: D1, D2, D3, J1, J2, J3, J4, R1, R2, R3
